Commit message: Started tuning urdf.

File: victoria_description/robots/victoria.xacro (robot description, xacro)
@@ -1,5 +1,5 @@
 <?xml version="1.0"?>
 <robot name="victoria_robot" xmlns:xacro="http://ros.org/wiki/xacro">
-  <xacro:arg name="laser_enabled" default="false" />
+  <xacro:arg name="laser_enabled" default="true" />
   <xacro:arg name="kinect_enabled" default="true" />
   <xacro:include filename="$(find victoria_description)/urdf/victoria.urdf.xacro" />

File: victoria_description/urdf/victoria.urdf.xacro (robot description, xacro)
@@ -15,8 +15,8 @@
   <xacro:property name="wheelbase" value="0.5120" />
   <xacro:property name="track" value="0.5708" />
-  <xacro:property name="wheel_vertical_offset" value="0.03282" />
+  <xacro:property name="wheel_vertical_offset" value="0.0" />
   <!-- Wheel Properties -->
   <xacro:property name="wheel_length" value="0.1143" />
-  <xacro:property name="wheel_radius" value="0.17775" />
+  <xacro:property name="wheel_radius" value="0.127" />
   <xacro:macro name="victoria_robot">
     <!-- Base link is the center of the robot's bottom plate -->
@@ -96,5 +96,5 @@
     <xacro:if value="$(arg kinect_enabled)">
       <xacro:sensor_arch prefix="" parent="top_plate_link">
-        <origin xyz="-0.25 0 0.41" rpy="0 0 -3.14"/>
+        <origin xyz="-0.25 -0.04 0.41" rpy="0 0.07 -3.14"/>
       </xacro:sensor_arch>
       <joint name="kinect_frame_joint" type="fixed">
