Commit message: Modified position for r200 for navigation

File: victoria_description/urdf/victoria.urdf.xacro (robot description, xacro)
@@ -23,5 +23,5 @@
     <link name="base_link">
       <visual>
-        <origin xyz="0 0 0" rpy="0 0 0" />
+        <origin xyz="0 0 ${base_z_size/2}" rpy="0 0 0" />
         <geometry>
           <mesh filename="package://victoria_description/meshes/base_link.dae" />
@@ -29,5 +29,5 @@
       </visual>
       <collision>
-        <origin xyz="0 0 ${base_z_size/4}" rpy="0 0 0" />
+        <origin xyz="0 0 ${base_z_size/2}" rpy="0 0 0" />
         <geometry>
           <box size="${base_x_size} ${base_y_size} ${base_z_size/2}"/>
@@ -35,5 +35,5 @@
       </collision>
       <collision>
-        <origin xyz="0 0 ${base_z_size*3/4}" rpy="0 0 0" />
+        <origin xyz="0 0 ${base_z_size/2}" rpy="0 0 0" />
         <geometry>
           <box size="${base_x_size*4/5} ${base_y_size} ${base_z_size/2}"/>
@@ -96,8 +96,8 @@
     <xacro:if value="$(arg kinect_enabled)">
       <xacro:sensor_arch prefix="" parent="top_plate_link">
-        <origin xyz="-0.35 0 0.51" rpy="0 0 -3.14"/>
+        <origin xyz="-0.25 0 0.41" rpy="0 0 -3.14"/>
       </xacro:sensor_arch>
       <joint name="kinect_frame_joint" type="fixed">
-        <origin xyz="0 0 0" rpy="0 0.18 3.14" />
+        <origin xyz="0 0 0" rpy="0 0. 3.14" />
         <parent link="sensor_arch_mount_link"/>
         <child link="camera_link"/>

Commit message: Updated the urdf and started breaking away from husky.

File: victoria_description/urdf/victoria.urdf.xacro (robot description, xacro)
@@ -4,7 +4,4 @@
   <xacro:include filename="$(find victoria_description)/urdf/decorations.urdf.xacro" />
   <xacro:include filename="$(find victoria_description)/urdf/wheel.urdf.xacro" />
-  <xacro:include filename="$(find victoria_description)/urdf/accessories/kinect_camera.urdf.xacro"/>
-  <xacro:include filename="$(find victoria_description)/urdf/accessories/sick_lms1xx_mount.urdf.xacro"/>
-  <xacro:include filename="$(find victoria_description)/urdf/accessories/sensor_arch.urdf.xacro"/>
   <xacro:property name="M_PI" value="3.14159"/>
   <!-- Base Size -->
@@ -13,7 +10,8 @@
   <xacro:property name="base_z_size" value="0.24750000" />
   <!-- Wheel Mounting Positions -->
-  <xacro:property name="wheelbase" value="0.5120" />
-  <xacro:property name="track" value="0.5708" />
-  <xacro:property name="wheel_vertical_offset" value="0.0" />
+  <xacro:property name="wheelbase" value="0.3" />
+  <xacro:property name="front_track" value="0.3" />
+  <xacro:property name="rear_track" value="0.47" />
+  <xacro:property name="wheel_vertical_offset" value="0.075" />
   <!-- Wheel Properties -->
   <xacro:property name="wheel_length" value="0.1143" />
@@ -44,5 +42,5 @@
     <link name="base_footprint"/>
     <joint name="base_footprint_joint" type="fixed">
-      <origin xyz="0 0 ${wheel_vertical_offset - wheel_radius}" rpy="0 0 0" />
+      <origin xyz="0 0 ${-wheel_radius}" rpy="0 0 0" />
       <parent link="base_link" />
       <child link="base_footprint" />
@@ -73,35 +71,46 @@
     <!-- Victoria wheel macros -->
     <xacro:victoria_wheel wheel_prefix="front_left">
-      <origin xyz="${wheelbase/2} ${track/2} ${wheel_vertical_offset}" rpy="0 0 0" />
+        <origin xyz="${wheelbase} ${front_track/2} ${-wheel_vertical_offset}" rpy="0 0 0" />
     </xacro:victoria_wheel>
     <xacro:victoria_wheel wheel_prefix="front_right">
-      <origin xyz="${wheelbase/2} ${-track/2} ${wheel_vertical_offset}" rpy="0 0 0" />
+        <origin xyz="${wheelbase} ${-front_track/2} ${-wheel_vertical_offset}" rpy="0 0 0" />
     </xacro:victoria_wheel>
     <xacro:victoria_wheel wheel_prefix="rear_left">
-      <origin xyz="${-wheelbase/2} ${track/2} ${wheel_vertical_offset}" rpy="0 0 0" />
+      <origin xyz="0.0 ${rear_track/2} 0.0" rpy="0 0 0" />
     </xacro:victoria_wheel>
     <xacro:victoria_wheel wheel_prefix="rear_right">
-      <origin xyz="${-wheelbase/2} ${-track/2} ${wheel_vertical_offset}" rpy="0 0 0" />
+      <origin xyz="0.0 ${-rear_track/2} 0.0" rpy="0 0 0" />
     </xacro:victoria_wheel>
     <xacro:victoria_decorate />
     <xacro:if value="$(arg laser_enabled)">
-      <sick_lms1xx_mount prefix="base" topic="scan"/>
+        <link name="laser_link">
+          <collision>
+            <origin xyz="0 0 .0585" rpy="0 0 0" />
+            <geometry>
+              <box size=".1 .108 .117" />
+            </geometry>
+          </collision>
+        </link>
       <joint name="laser_mount_joint" type="fixed">
-        <origin xyz="0.2206 0.0 0.00635"
+        <origin xyz="0.27 0.0 0.1"
                 rpy="0.0 0.0 0.0" />
-        <parent link="top_plate_link" />
-        <child link="base_laser_mount" />
+        <parent link="base_link" />
+        <child link="laser_link" />
       </joint>
     </xacro:if>
     <xacro:if value="$(arg kinect_enabled)">
-      <xacro:sensor_arch prefix="" parent="top_plate_link">
-        <origin xyz="-0.25 -0.04 0.41" rpy="0 0.07 -3.14"/>
-      </xacro:sensor_arch>
-      <joint name="kinect_frame_joint" type="fixed">
-        <origin xyz="0 0 0" rpy="0 0. 3.14" />
-        <parent link="sensor_arch_mount_link"/>
+        <link name="camera_link">
+          <collision>
+            <origin xyz="0 0 .0585" rpy="0 0 0" />
+            <geometry>
+              <box size=".1 .108 .117" />
+            </geometry>
+          </collision>
+        </link>
+      <joint name="r200_frame_joint" type="fixed">
+        <origin xyz="-0.17 -0.04 0.26" rpy="0.0 -0.087 0.0" />
+        <parent link="base_link"/>
         <child link="camera_link"/>
       </joint>
-      <xacro:kinect_camera prefix="camera"/>
     </xacro:if>
   </xacro:macro>

Commit message: Started tweaking the imu link.

File: victoria_description/urdf/victoria.urdf.xacro (robot description, xacro)
@@ -63,5 +63,5 @@
     <link name="imu_link"/>
     <joint name="imu_joint" type="fixed">
-      <origin xyz="0.19 0 0.149" rpy="0 -1.5708 3.1416" />
+      <origin xyz="0 0 0" rpy="0 0 -3.1416" />
       <parent link="base_link" />
       <child link="imu_link" />

Commit message: Added gps link.

File: victoria_description/urdf/victoria.urdf.xacro (robot description, xacro)
@@ -69,4 +69,12 @@
     <gazebo reference="imu_link">
     </gazebo>
+    <link name="gps"/>
+    <joint name="gps_joint" type="fixed">
+      <origin xyz="0 0 0" rpy="0 0 0" />
+      <parent link="base_link" />
+      <child link="gps" />
+    </joint>
+    <gazebo reference="gps">
+    </gazebo>
     <!-- Victoria wheel macros -->
     <xacro:victoria_wheel wheel_prefix="front_left">

Commit message: Rotated yaw back by 90 degrees to get things to point in the same direction.

File: victoria_description/urdf/victoria.urdf.xacro (robot description, xacro)
@@ -63,5 +63,5 @@
     <link name="imu_link"/>
     <joint name="imu_joint" type="fixed">
-      <origin xyz="0 0 0" rpy="0 0 -3.1416" />
+        <origin xyz="0 0 0" rpy="0 0 -3.1416/2" />
       <parent link="base_link" />
       <child link="imu_link" />
